File: DualChannel_PowerSwitch_Low.kicad_pcb (KiCad board)
At the start: 2 copper layers, 33 x 38.1 mm, 14 parts, among them J1 Conn_01x04, J2 Conn_01x04, M1 SCREW_6-32_POWER, M2 SCREW_6-32_POWER, M4 SCREW_6-32_POWER, M5 SCREW_6-32_POWER, M6 SCREW_6-32_POWER, M7 SCREW_6-32_POWER, Q1 INFINEON_IRLML0040TRPBF, Q2 INFINEON_IRLML0040TRPBF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

Commit message: Adjusted header position slightly
Parts:
- moved J2 1.78 mm to (177.8, 114.3)
Changed lines of the file:
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@@
   )
   (setup
-    (last_trace_width 0.508)
+    (last_trace_width 0.25)
     (user_trace_width 0.381)
     (user_trace_width 0.508)
@@
     (mod_text_size 1 1)
     (mod_text_width 0.15)
-    (pad_size 1.524 1.524)
-    (pad_drill 0.762)
+    (pad_size 1.7 1.7)
+    (pad_drill 1)
     (pad_to_mask_clearance 0.051)
     (solder_mask_min_width 0.25)
     (aux_axis_origin 0 0)
     (grid_origin 183.388 131.318)
-    (visible_elements FFFFFF7F)
+    (visible_elements 7FFFFFFF)
     (pcbplotparams
       (layerselection 0x010fc_ffffffff)
@@
   )
   (module Pin_Headers:Pin_Header_Straight_1x04_Pitch2.54mm (layer F.Cu)
-    (at 176.022 114.3)
+    (at 177.8 114.3)
     (descr "Through hole straight pin header, 1x04, 2.54mm pitch, single row")
     (tags "Through hole pin header THT 1x04 2.54mm single row")
